Commit message: Made sensor and user rails as args toggleable.

File: husky_description/urdf/decorations.urdf.xacro (robot description, xacro)
@@ -11,4 +11,6 @@
     <xacro:property name="husky_front_bumper_extend" value="$(optenv HUSKY_FRONT_BUMPER_EXTEND 0)" />
     <xacro:property name="husky_rear_bumper_extend" value="$(optenv HUSKY_REAR_BUMPER_EXTEND 0)" />
+    <xacro:arg name="user_rail_enabled" default="$(optenv HUSKY_USER_RAIL_ENABLED 1)" />
+    <xacro:arg name="sensor_rail_enabled" default="$(optenv HUSKY_SENSOR_RAIL_ENABLED 1)" />
     <!-- Spawn Husky chassis -->
     <link name="top_chassis_link">
@@ -25,5 +27,5 @@
       <child link="top_chassis_link" />
     </joint>
-    <xacro:if value="$(optenv HUSKY_USER_RAIL_ENABLED true)">
+    <xacro:if value="$(arg user_rail_enabled)">
       <!-- Spawn user rails -->
       <link name="user_rail_link">
@@ -170,4 +172,10 @@
       <link name="top_plate_rear_link"/>
     </xacro:if>
+    <!-- Sensor Rail -->
+    <xacro:if value="$(arg sensor_rail_enabled)">
+      <xacro:sensor_arch prefix="" parent="top_plate_link">
+        <origin xyz="-0.35 0 0.51" rpy="0 0 -3.14"/>
+      </xacro:sensor_arch>
+    </xacro:if>
   </xacro:macro>
 </robot>

File: husky_description/urdf/husky_macro.urdf.xacro (robot description, xacro)
@@ -4,5 +4,5 @@
   <xacro:arg name="laser_xyz" default="$(optenv CPR_LASER_XYZ 0.2206 0.0 0.00635)" />
   <xacro:arg name="laser_rpy" default="$(optenv CPR_LASER_RPY 0.0 0.0 0.0)" />
-  <xacro:arg name="realsense_enabled" default="$(optenv CPR_REALSENSE 0)" />
+  <xacro:arg name="realsense_enabled" default="$(optenv CPR_REALSENSE 1)" />
   <xacro:arg name="realsense_xyz" default="$(optenv CPR_REALSENSE_XYZ 0 0 0)" />
   <xacro:arg name="realsense_rpy" default="$(optenv CPR_REALSENSE_RPY 0 0 0)" />
@@ -113,16 +113,5 @@
       </joint>
     </xacro:if>
-    <!--
-      top sensor arch; include this if we have realsense enabled
-      keep this as a property to make it easier to add multiple conditions, should we need
-      the top bar for any additional sensors in the future
-    -->
-    <!-- <xacro:property name="topbar_needed_realsense" value="$(arg realsense_enabled)" />
-    <xacro:if value="${topbar_needed_realsense}">
-      <xacro:sensor_arch prefix="" parent="top_plate_link">
-        <origin xyz="-0.35 0 0.51" rpy="0 0 -3.14"/>
-      </xacro:sensor_arch>
-    </xacro:if> -->
-    <!-- add the intel realsense to the topbar if needed -->
+    <!-- add the intel realsense to the topbar if needed
     <xacro:if value="$(arg realsense_enabled)">
       <link name="realsense_mountpoint"/>
@@ -134,4 +123,5 @@
       <xacro:intel_realsense_mount prefix="camera" topic="realsense" parent_link="realsense_mountpoint"/>
     </xacro:if>
+    -->
     <ros2_control name="${prefix}husky_hardware" type="system">
       <hardware>
